Commit message: dart: flatten the model directory hierarchy a bit.

File: src/dart/urdf/iiwa14_simple.urdf (robot description, URDF)
Before this commit: robot iiwa14, 10 links, 9 joints
Links:
- link iiwa_link_0: geometry collision box size=0.24 0.23 0.1575; visual mesh filename=package://iiwa14/link_0.stl
- link iiwa_link_1: geometry collision box size=0.175 0.19 0.26; visual mesh filename=package://iiwa14/link_1.stl
- link iiwa_link_2: geometry collision box size=0.175 0.24 0.19; visual mesh filename=package://iiwa14/link_2.stl
- link iiwa_link_3: geometry collision box size=0.125 0.15 0.26; visual mesh filename=package://iiwa14/link_3.stl
- link iiwa_link_4: geometry collision box size=0.125 0.22 0.15; visual mesh filename=package://iiwa14/link_4.stl
- link iiwa_link_5: geometry collision box size=0.125 0.15 0.24; visual mesh filename=package://iiwa14/link_5.stl
- link iiwa_link_6: geometry collision box size=0.125 0.15 0.125; visual mesh filename=package://iiwa14/link_6.stl
- link iiwa_link_7: geometry collision box size=0.1 0.1 0.05; visual mesh filename=package://iiwa14/link_7.stl

File: src/dart/urdf/robotiq.urdf (robot description, URDF)
Before this commit: robot robotiq_arg85_description, 9 links, 8 joints
Links:
- link left_inner_finger: geometry collision box size=0.015 0.03 0.05; visual mesh filename=package://robotiq/inner_finger_fine.stl
- link left_inner_knuckle: geometry visual mesh filename=package://robotiq/inner_knuckle_fine.stl
- link left_outer_finger: geometry collision box size=0.01 0.03 0.06; visual mesh filename=package://robotiq/outer_finger_fine.stl
- link left_outer_knuckle: geometry visual mesh filename=package://robotiq/outer_knuckle_fine.stl
- link right_inner_finger: geometry collision box size=0.015 0.03 0.05; visual mesh filename=package://robotiq/inner_finger_fine.stl
- link right_inner_knuckle: geometry visual mesh filename=package://robotiq/inner_knuckle_fine.stl
- link right_outer_finger: geometry collision box size=0.01 0.03 0.06; visual mesh filename=package://robotiq/outer_finger_fine.stl
- link right_outer_knuckle: geometry visual mesh filename=package://robotiq/outer_knuckle_fine.stl
- link robotiq_85_base_link: geometry collision box size=0.07 0.07 0.09; visual mesh filename=package://robotiq/robotiq_85_base_link_fine.stl
